File: eagle/midi_to_cv.brd (EAGLE design)
At the start: 100.3 x 80 mm, 36 parts, among them IC1 TL074P, IC4 TL074P, IC5 TL074P, U1 ATMEGA328P_PDIP

Commit message: routed
Parts:
- added C10, C12, C8: 100n, rcl:C025-024X044
- added R12, R20, R29, R32, R34, R35, R36, R37, R38, R39, R40, R41, R43: 1k, rcl:0204/7
- added R13, R14, R16, R19, R21, R23, R28, R30, R31, R33, R42: 1k, rcl:0204/5
- added R17, R18, R24, R25, R26, R27: 1k8, rcl:0204V
- added X1, X2: (no value), con-molex:KK-156-6
- R10, R9: device rcl:0207/10 -> rcl:0204V
- R11, R3, R8: value 1k -> 1k8; device rcl:0207/10 -> rcl:0204V
- R5: device rcl:0207/10 -> rcl:0204/7
- R7: value 6k8 -> 1k8; device rcl:0207/10 -> rcl:0204V
- moved R10 185.1 mm to (53.3, 71.1), turned to 90 degrees
- moved R9 183.9 mm to (66.0, 71.1), turned to 90 degrees
- moved R11 177.8 mm to (53.3, 58.4), turned to 270 degrees
- moved R8 167.2 mm to (66.0, 58.4), turned to 270 degrees
- moved R3 165.6 mm to (88.9, 55.9)
- moved R7 164.2 mm to (76.2, 55.9), turned to 180 degrees
- moved R2 158.2 mm to (21.6, 74.9)
- moved MIDI_OUT_THRU1 148.9 mm to (33.0, 72.4)
- moved IC4 109.8 mm to (82.5, 49.5), turned to 180 degrees
- moved IC5 93.0 mm to (59.7, 33.0), turned to 270 degrees
- moved PWR1 92.7 mm to (22.9, 6.35), turned to 180 degrees
- moved C7 84.3 mm to (4.45, 17.8), turned to 270 degrees
- moved C5 82.8 mm to (8.26, 17.8), turned to 270 degrees
- moved U$5 82.7 mm to (12.2, 17.1), turned to 90 degrees
- moved U$4 81.0 mm to (17.0, 17.1), turned to 90 degrees
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Connections:
- removed net V+: IC1.4, IC4.4, IC5.4
- removed net V-: IC1.11, IC4.11, IC5.11
- new net N$24: IC4.9, R17.1, R19.2
- new net N$25: R34.2, X1.1
- new net N$26: IC1.3, U$1.2
- new net N$27: IC1.5, U$1.3
- new net N$28: IC1.10, U$1.4
- new net N$29: IC1.12, U$1.5
- new net N$30: IC4.6, R20.2, R7.1
- new net N$31: IC4.2, R21.2, R3.1
- new net N$32: IC4.5, U$1.6
- new net N$33: IC4.3, U$1.7
- new net N$34: IC4.12, U$1.14
- new net N$35: IC4.10, U$1.15
- new net N$36: IC4.13, R18.1, R23.2
- new net N$37: IC4.1, R3.2, R37.1
- new net N$38: R35.2, X1.2
- new net N$39: R33.2, X1.3
- new net N$40: R32.2, X1.4
- new net N$41: IC5.3, U$1.16
- new net N$42: IC5.5, U$1.17
- new net N$43: IC5.10, U$1.18
- new net N$44: IC5.12, U$1.19
- new net N$45: IC5.2, R24.1, R28.2
- new net N$46: IC5.6, R25.1, R29.2
- new net N$47: IC5.9, R26.1, R30.2
- new net N$48: IC5.13, R27.1, R31.2
- new net N$49: IC5.1, R24.2, R40.1
- new net N$50: IC5.7, R25.2, R41.1
- new net N$51: IC5.8, R26.2, R42.1
- new net N$52: IC5.14, R27.2, R43.1
- new net N$53: IC1.1, R32.1, R8.2
- new net N$54: IC1.7, R33.1, R9.2
- new net N$55: IC1.8, R10.2, R34.1
- new net N$56: IC1.14, R11.2, R35.1
- new net N$57: R36.2, X1.5
- new net N$58: R37.2, X1.6
- new net N$59: R40.2, X2.1
- new net N$61: R41.2, X2.2
- new net N$63: R42.2, X2.3
- new net N$64: R43.2, X2.4
- new net N$65: R39.2, X2.5
- new net N$66: R38.2, X2.6
- net +12V: now also C10.1, C12.1, C8.1, IC1.4, IC4.4, IC5.4
- net +5V: no longer R7.2
- net GND: now also C10.2, C12.2, C8.2, IC1.11, IC4.11, IC5.11, R12.1, R13.1, R14.1, R16.1, R19.1, R20.1, R21.1, R23.1, R28.1, R29.1, R30.1, R31.1; no longer R11.1, R3.1, R8.1
- net N$13: now also R12.2, R8.1; no longer IC1.9, R3.2, R7.1
- net N$14: now also IC1.9, R10.1, R14.2; no longer IC1.3, IC1.5, U$1.2
- net N$15: now also R13.2; no longer R8.2
- net N$16: now also IC4.7, R36.1, R7.2; no longer IC1.7, R9.2
- net N$21: now also R11.1, R16.2; no longer R10.1, R11.2
- net N$22: now also IC4.8, R17.2, R39.1; no longer IC1.10, U$1.3
- net N$23: now also IC4.14, R18.2, R38.1; no longer IC1.14, R10.2
Routing:
- net GND: track 0.00 -> 375.1 mm, vias 0 -> 2
- net +5V: track 0.00 -> 249.5 mm, vias 0 -> 6
- net +12V: track 0.00 -> 185.2 mm, vias 0 -> 2
- net N$38: track 0.00 -> 52.3 mm
- net N$34: track 0.00 -> 39.8 mm
- net N$33: track 0.00 -> 39.1 mm
- net N$25: track 0.00 -> 36.8 mm
- net N$32: track 0.00 -> 29.9 mm
- net N$35: track 0.00 -> 29.9 mm
- net N$66: track 0.00 -> 27.9 mm
- net N$17: track 0.00 -> 24.3 mm
- net N$57: track 0.00 -> 22.4 mm
- net N$59: track 0.00 -> 22.1 mm
- net N$40: track 0.00 -> 20.9 mm
- net N$8: track 0.00 -> 19.7 mm
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Other:
- outline, holes or cut-outs redrawn

Commit message: tweaks
Parts:
- R29, R35, R41: device rcl:0204/7 -> rcl:0204/5
- moved PAD13 4.89 mm to (14.7, 30.7)
- moved R29 4.32 mm to (50.8, 27.2)
- moved R2 4.06 mm to (21.6, 70.9)
- moved PWR1 3.94 mm to (26.7, 5.33)
- moved R35 3.81 mm to (44.5, 59.7)
- moved R34 3.59 mm to (46.5, 68.8)
- moved R33 3.57 mm to (71.4, 68.8)
- moved MIDI_IN 3.56 mm to (12.1, 67.6)
- moved R1 3.56 mm to (21.6, 67.6)
- moved R10 3.56 mm to (53.3, 67.6)
- moved R9 3.56 mm to (66.0, 67.6)
- moved C1 3.56 mm to (20.3, 46.0)
- moved C10 3.56 mm to (53.3, 29.5)
- moved C8 3.56 mm to (83.8, 52.3)
- moved IC4 3.56 mm to (82.5, 46.0)
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Routing:
- net +5V: track 249.5 -> 243.7 mm
- net +12V: track 185.2 -> 181.3 mm
- net N$62: track 11.2 -> 14.7 mm
- net N$2: track 10.1 -> 12.9 mm
- net GND: track 375.1 -> 373.2 mm
- net N$38: track 52.3 -> 54.1 mm
- net N$61: track 12.4 -> 13.5 mm
- net N$63: track 12.8 -> 11.8 mm
- net N$55: track 5.08 -> 5.59 mm
Other:
- outline, holes or cut-outs redrawn
